File: LayoutPCB.kicad_pcb (KiCad board)
At the start: 2 copper layers, 59.2 x 48.9 mm, 39 parts, among them J1 USB_B_Micro, J2 Conn_01x01_Female, J3 Conn_01x01_Female, J4 Conn_01x01_Female, J5 Conn_01x01_Female, J6 Conn_01x01_Female, J7 Conn_01x01_Female, U1 TP4056, U2 DW01, U3 FS8205A

Commit message: Adicionando os conectores
Parts:
- removed the REF** at (83.9, 39.3)
- added ?: , , F.Cu at (64.4, 58.0)
- added REF**: PinSocket_1x01_P2.54mm_Vertical, Connector_PinSocket_2.54mm:PinSocket_1x01_P2.54mm_Vertical, F.Cu at (65.0, 71.8)
- added REF**: PinSocket_1x01_P2.54mm_Vertical, Connector_PinSocket_2.54mm:PinSocket_1x01_P2.54mm_Vertical, F.Cu at (108.5, 61.3)
- added REF**: PinSocket_1x01_P2.54mm_Vertical, Connector_PinSocket_2.54mm:PinSocket_1x01_P2.54mm_Vertical, F.Cu at (108.6, 66.7)
- added REF**: PinSocket_1x01_P2.54mm_Vertical, Connector_PinSocket_2.54mm:PinSocket_1x01_P2.54mm_Vertical, F.Cu at (108.3, 57.0)
- added REF**: PinSocket_1x01_P2.54mm_Vertical, Connector_PinSocket_2.54mm:PinSocket_1x01_P2.54mm_Vertical, F.Cu at (108.5, 71.2)
- added REF**: DHT22, Connector_PinSocket_2.54mm:PinSocket_1x04_P2.54mm_Vertical, F.Cu at (83.9, 38.9)
Routing:
- net GND: track 108.9 -> 226.4 mm, vias 0 -> 1
- net (no net): track 1037.3 -> 949.7 mm, vias 14 -> 7
Other:
- board text added: "Placa de Sensor de Temperatua e Umidade ESP 32 com Lora, display OLED e Bateria Revisão 1.0 Autor Rafael Pascale"
- board text removed: "Placa de Sensor de Temperatua e Umidade ESP 32 com Lora e display OLED e Bateria Revisão 1.0 Autor Rafael Pascale"
